Commit message: 4.12初始备份

File: smart_pick_and_place_ws/src/rm_description/urdf/SingleArm/easy_single_arm.urdf (robot description, URDF)
Before this commit: robot rm_65_description, 25 links, 24 joints
Joints:
- joint L_hand_joint_endeffector: origin xyz=0.020 -0.051 -0.156 rpy=2.222 0 0.05 -> xyz=0.030 -0.053 -0.15 rpy=2.222 0 0.05
