Commit message: 部分动作录制，联合标定脚本上传，实现两臂轻量联动递物拆解

File: dependence/smart_pick_and_place_ws/src/rm_description/urdf/LeftArm/right_arm.urdf (robot description, URDF)
Before this commit: robot rm_65_right_description, 14 links, 13 joints
Links:
- added link R_left_inner_finger, mass 0.00724255346165745; collision mesh filename=package://rm_description/meshes/singlearm/robotiq_85/inner_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; visual mesh filename=package://rm_description/meshes/singlearm/robotiq_85/inner_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
- added link R_left_inner_knuckle, mass 0.0110930853895903; collision mesh filename=package://rm_description/meshes/singlearm/robotiq_85/inner_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; visual mesh filename=package://rm_description/meshes/singlearm/robotiq_85/inner_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
- added link R_left_outer_finger, mass 0.0273093985570947; collision mesh filename=package://rm_description/meshes/singlearm/robotiq_85/outer_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; visual mesh filename=package://rm_description/meshes/singlearm/robotiq_85/outer_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
- added link R_left_outer_knuckle, mass 0.00684838849434396; collision mesh filename=package://rm_description/meshes/singlearm/robotiq_85/outer_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; visual mesh filename=package://rm_description/meshes/singlearm/robotiq_85/outer_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
- added link R_right_inner_finger, mass 0.00724255346165744; collision mesh filename=package://rm_description/meshes/singlearm/robotiq_85/inner_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; visual mesh filename=package://rm_description/meshes/singlearm/robotiq_85/inner_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
- added link R_right_inner_knuckle, mass 0.0110930853895903; collision mesh filename=package://rm_description/meshes/singlearm/robotiq_85/inner_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; visual mesh filename=package://rm_description/meshes/singlearm/robotiq_85/inner_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
- added link R_right_outer_finger, mass 0.0273093985570947; collision mesh filename=package://rm_description/meshes/singlearm/robotiq_85/outer_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; visual mesh filename=package://rm_description/meshes/singlearm/robotiq_85/outer_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
- added link R_right_outer_knuckle, mass 0.00684838849401352; collision mesh filename=package://rm_description/meshes/singlearm/robotiq_85/outer_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; visual mesh filename=package://rm_description/meshes/singlearm/robotiq_85/outer_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
- link R_gripper_base: mass 0.3 -> 0.30915; geometry collision mesh filename=package://rm_description/meshes/singlearm/robotiq_85/roboti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; visual mesh filename=package://rm_description/meshes/singlearm/robotiq_85/roboti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
Joints:
- added joint R_finger_joint: type revolute, parent R_gripper_base, child R_left_outer_knuckle, origin xyz=0.0306011444260539 0 0.0627920162695395 rpy=0 0 0, axis 0 -1 0, limit lower=0 upper=0.725 effort=1000 velocity=2.0
- added joint R_left_inner_finger_joint: type revolute, parent R_left_inner_knuckle, child R_left_inner_finger, origin xyz=0.034585310861294 0 0.0454970193817975 rpy=0 0 0, axis 0 -1 0, limit lower=0 upper=0.8757 effort=1000 velocity=2.0, mimic joint=R_finger_joint multiplier=-1 offset=0
- added joint R_left_inner_knuckle_joint: type revolute, parent R_gripper_base, child R_left_inner_knuckle, origin xyz=0.0127000000001501 0 0.0693074999999639 rpy=0 0 0, axis 0 -1 0, limit lower=0 upper=0.8757 effort=1000 velocity=2.0, mimic joint=R_finger_joint multiplier=1 offset=0
- added joint R_left_outer_finger_joint: type fixed, parent R_left_outer_knuckle, child R_left_outer_finger, origin xyz=0.0316910442266543 0 -0.00193396375724605 rpy=0 0 0, axis 0 -1 0
- added joint R_right_inner_finger_joint: type revolute, parent R_right_inner_knuckle, child R_right_inner_finger, origin xyz=0.0341060475457406 0 0.0458573878541688 rpy=0 0 0, axis 0 1 0, limit lower=0 upper=0.8757 effort=1000 velocity=2.0, mimic joint=R_finger_joint multiplier=1 offset=0
- added joint R_right_inner_knuckle_joint: type revolute, parent R_gripper_base, child R_right_inner_knuckle, origin xyz=-0.0126999999998499 0 0.0693075000000361 rpy=0 0 3.14159265358979, axis 0 1 0, limit lower=0 upper=0.8757 effort=1000 velocity=2.0, mimic joint=R_finger_joint multiplier=-1 offset=0
- added joint R_right_outer_finger_joint: type fixed, parent R_right_outer_knuckle, child R_right_outer_finger, origin xyz=0.0317095909367246 0 -0.0016013564954687 rpy=0 0 0, axis 0 1 0
- added joint R_right_outer_knuckle_joint: type revolute, parent R_gripper_base, child R_right_outer_knuckle, origin xyz=-0.0306011444258893 0 0.0627920162695395 rpy=0 0 3.14159265358979, axis 0 1 0, limit lower=0 upper=0.8757 effort=1000 velocity=2.0, mimic joint=R_finger_joint multiplier=-1 offset=0
- joint R_arm_to_gripper: origin xyz=0 0 0.01 rpy=0 3.1416 -1.5708 -> xyz=0 0 0.01 rpy=0 0 1.5708
- joint R_gripper_endeffector_joint: origin xyz=0 0 -0.10 rpy=0 0 0 -> xyz=0 0 0.15 rpy=0 0 0
