Commit message: feat: implement SimServer RGB-D camera rendering + camera link

File: dependence/smart_pick_and_place_ws/src/rm_description/urdf/left_arm_bullet.urdf (robot description, URDF)
Before this commit: robot rm_65_description, 21 links, 20 joints
Links:
- added link cam_link_grasp
Joints:
- added joint cam_link_grasp_joint: type fixed, parent Link7, child cam_link_grasp, origin xyz=0.0 0.0 0.0 rpy=0 0 0
