Commit message: debug: 扁平化 URDF 目录结构 + 清理右臂占位姿
- meshes/singlearm/{rm75_6f,robotiq_85,inspire_hand} → meshes/（原命名误指单臂，实为机械臂+夹爪+灵巧手所有 mesh）
- urdf/LeftArm/{left,right}_arm*.urdf → urdf/（原命名误指左臂，实含左右两臂 urdf）
- 同步更新 4 个 urdf 中 168 处 mesh 路径引用
- 同步更新 bringup.launch / twin.py / inspire_hand_bringup.py 中 URDF 路径
- 删除 robot_config.json 中 4 个全 0 占位姿：arms.right.desk_pose_1/2/3、dual_arm.show_to_camera

File: dependence/smart_pick_and_place_ws/src/rm_description/urdf/dual_arm.urdf (robot description, URDF)
Before this commit: robot dual_arm, 53 links, 52 joints
Links:
- link L_hand_base_link: geometry collision mesh filename=package://rm_description/meshes/inspire_hand/l_base_link.STL; visual mesh filename=package://rm_description/meshes/inspire_hand/l_base_link.STL
- link Link1: geometry collision mesh filename=package://rm_description/meshes/rm75_6f/link1_l.STL; visual mesh filename=package://rm_description/meshes/rm75_6f/link1_l.STL
- link Link2: geometry collision mesh filename=package://rm_description/meshes/rm75_6f/link2_l.STL; visual mesh filename=package://rm_description/meshes/rm75_6f/link2_l.STL
- link Link3: geometry collision mesh filename=package://rm_description/meshes/rm75_6f/link3_l.STL; visual mesh filename=package://rm_description/meshes/rm75_6f/link3_l.STL
- link Link4: geometry collision mesh filename=package://rm_description/meshes/rm75_6f/link4_l.STL; visual mesh filename=package://rm_description/meshes/rm75_6f/link4_l.STL
- link Link5: geometry collision mesh filename=package://rm_description/meshes/rm75_6f/link5_l.STL; visual mesh filename=package://rm_description/meshes/rm75_6f/link5_l.STL
- link Link6: geometry collision mesh filename=package://rm_description/meshes/rm75_6f/link6_l.STL; visual mesh filename=package://rm_description/meshes/rm75_6f/link6_l.STL
- link Link7: geometry collision mesh filename=package://rm_description/meshes/rm75_6f/link7_l.STL; visual mesh filename=package://rm_description/meshes/rm75_6f/link7_l.STL
- link R_Link1: geometry collision mesh filename=package://rm_description/meshes/rm75_6f/link1_l.STL; visual mesh filename=package://rm_description/meshes/rm75_6f/link1_l.STL
- link R_Link2: geometry collision mesh filename=package://rm_description/meshes/rm75_6f/link2_l.STL; visual mesh filename=package://rm_description/meshes/rm75_6f/link2_l.STL
- link R_Link3: geometry collision mesh filename=package://rm_description/meshes/rm75_6f/link3_l.STL; visual mesh filename=package://rm_description/meshes/rm75_6f/link3_l.STL
- link R_Link4: geometry collision mesh filename=package://rm_description/meshes/rm75_6f/link4_l.STL; visual mesh filename=package://rm_description/meshes/rm75_6f/link4_l.STL
- link R_Link5: geometry collision mesh filename=package://rm_description/meshes/rm75_6f/link5_l.STL; visual mesh filename=package://rm_description/meshes/rm75_6f/link5_l.STL
- link R_Link6: geometry collision mesh filename=package://rm_description/meshes/rm75_6f/link6_l.STL; visual mesh filename=package://rm_description/meshes/rm75_6f/link6_l.STL
- link R_Link7: geometry collision mesh filename=package://rm_description/meshes/rm75_6f/link7_l.STL; visual mesh filename=package://rm_description/meshes/rm75_6f/link7_l.STL
- link R_gripper_base: geometry collision mesh filename=package://rm_description/meshes/robotiq_85/robotiq_85_base_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; visual mesh filename=package://rm_description/meshes/robotiq_85/robotiq_85_base_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
- link R_left_inner_finger: geometry collision mesh filename=package://rm_description/meshes/robotiq_85/inner_finger_coa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; visual mesh filename=package://rm_description/meshes/robotiq_85/inner_finger_fin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
- link R_left_inner_knuckle: geometry collision mesh filename=package://rm_description/meshes/robotiq_85/inner_knuckle_co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; visual mesh filename=package://rm_description/meshes/robotiq_85/inner_knuckle_fi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
- link R_left_outer_finger: geometry collision mesh filename=package://rm_description/meshes/robotiq_85/outer_finger_coa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; visual mesh filename=package://rm_description/meshes/robotiq_85/outer_finger_fin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
- link R_left_outer_knuckle: geometry collision mesh filename=package://rm_description/meshes/robotiq_85/outer_knuckle_co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; visual mesh filename=package://rm_description/meshes/robotiq_85/outer_knuckle_fi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
- link R_right_inner_finger: geometry collision mesh filename=package://rm_description/meshes/robotiq_85/inner_finger_coa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; visual mesh filename=package://rm_description/meshes/robotiq_85/inner_finger_fin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
- link R_right_inner_knuckle: geometry collision mesh filename=package://rm_description/meshes/robotiq_85/inner_knuckle_co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; visual mesh filename=package://rm_description/meshes/robotiq_85/inner_knuckle_fi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
- link R_right_outer_finger: geometry collision mesh filename=package://rm_description/meshes/robotiq_85/outer_finger_coa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; visual mesh filename=package://rm_description/meshes/robotiq_85/outer_finger_fin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
- link R_right_outer_knuckle: geometry collision mesh filename=package://rm_description/meshes/robotiq_85/outer_knuckle_co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; visual mesh filename=package://rm_description/meshes/robotiq_85/outer_knuckle_fi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
- link R_robot_base_link: geometry collision mesh filename=package://rm_description/meshes/rm75_6f/base_link_l.STL; visual mesh filename=package://rm_description/meshes/rm75_6f/base_link_l.STL
- link left_index_1: geometry collision mesh filename=package://rm_description/meshes/inspire_hand/left_index_1.S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; visual mesh filename=package://rm_description/meshes/inspire_hand/left_index_1.S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
- link left_index_2: geometry collision mesh filename=package://rm_description/meshes/inspire_hand/left_index_2.S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; visual mesh filename=package://rm_description/meshes/inspire_hand/left_index_2.S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
- link left_little_1: geometry collision mesh filename=package://rm_description/meshes/inspire_hand/left_little_1.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; visual mesh filename=package://rm_description/meshes/inspire_hand/left_little_1.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
- link left_little_2: geometry collision mesh filename=package://rm_description/meshes/inspire_hand/left_little_2.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; visual mesh filename=package://rm_description/meshes/inspire_hand/left_little_2.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
- link left_middle_1: geometry collision mesh filename=package://rm_description/meshes/inspire_hand/left_middle_1.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; visual mesh filename=package://rm_description/meshes/inspire_hand/left_middle_1.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
- link left_middle_2: geometry collision mesh filename=package://rm_description/meshes/inspire_hand/left_middle_2.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; visual mesh filename=package://rm_description/meshes/inspire_hand/left_middle_2.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
- link left_ring_1: geometry collision mesh filename=package://rm_description/meshes/inspire_hand/left_ring_1.STL; visual mesh filename=package://rm_description/meshes/inspire_hand/left_ring_1.STL
- link left_ring_2: geometry collision mesh filename=package://rm_description/meshes/inspire_hand/left_ring_2.STL; visual mesh filename=package://rm_description/meshes/inspire_hand/left_ring_2.STL
- link left_thumb_1: geometry collision mesh filename=package://rm_description/meshes/inspire_hand/left_thumb_1.S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; visual mesh filename=package://rm_description/meshes/inspire_hand/left_thumb_1.S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
- link left_thumb_2: geometry collision mesh filename=package://rm_description/meshes/inspire_hand/left_thumb_2.S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; visual mesh filename=package://rm_description/meshes/inspire_hand/left_thumb_2.S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
- link left_thumb_3: geometry collision mesh filename=package://rm_description/meshes/inspire_hand/left_thumb_3.S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; visual mesh filename=package://rm_description/meshes/inspire_hand/left_thumb_3.S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
- link left_thumb_swing: geometry collision mesh filename=package://rm_description/meshes/inspire_hand/left_thumb_swi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; visual mesh filename=package://rm_description/meshes/inspire_hand/left_thumb_swi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
- link robot_base_link: geometry collision mesh filename=package://rm_description/meshes/rm75_6f/base_link_l.STL; visual mesh filename=package://rm_description/meshes/rm75_6f/base_link_l.STL

File: dependence/smart_pick_and_place_ws/src/rm_description/urdf/left_arm.urdf (robot description, URDF)
Before this commit: robot rm_65_description, 25 links, 24 joints
Links:
- link L_hand_base_link: geometry collision mesh filename=package://rm_description/meshes/inspire_hand/l_base_link.STL; visual mesh filename=package://rm_description/meshes/inspire_hand/l_base_link.STL
- link Link1: geometry collision mesh filename=package://rm_description/meshes/rm75_6f/link1_l.STL; visual mesh filename=package://rm_description/meshes/rm75_6f/link1_l.STL
- link Link2: geometry collision mesh filename=package://rm_description/meshes/rm75_6f/link2_l.STL; visual mesh filename=package://rm_description/meshes/rm75_6f/link2_l.STL
- link Link3: geometry collision mesh filename=package://rm_description/meshes/rm75_6f/link3_l.STL; visual mesh filename=package://rm_description/meshes/rm75_6f/link3_l.STL
- link Link4: geometry collision mesh filename=package://rm_description/meshes/rm75_6f/link4_l.STL; visual mesh filename=package://rm_description/meshes/rm75_6f/link4_l.STL
- link Link5: geometry collision mesh filename=package://rm_description/meshes/rm75_6f/link5_l.STL; visual mesh filename=package://rm_description/meshes/rm75_6f/link5_l.STL
- link Link6: geometry collision mesh filename=package://rm_description/meshes/rm75_6f/link6_l.STL; visual mesh filename=package://rm_description/meshes/rm75_6f/link6_l.STL
- link Link7: geometry collision mesh filename=package://rm_description/meshes/rm75_6f/link7_l.STL; visual mesh filename=package://rm_description/meshes/rm75_6f/link7_l.STL
- link left_index_1: geometry collision mesh filename=package://rm_description/meshes/inspire_hand/left_index_1.S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; visual mesh filename=package://rm_description/meshes/inspire_hand/left_index_1.S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
- link left_index_2: geometry collision mesh filename=package://rm_description/meshes/inspire_hand/left_index_2.S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; visual mesh filename=package://rm_description/meshes/inspire_hand/left_index_2.S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
- link left_little_1: geometry collision mesh filename=package://rm_description/meshes/inspire_hand/left_little_1.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; visual mesh filename=package://rm_description/meshes/inspire_hand/left_little_1.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
- link left_little_2: geometry collision mesh filename=package://rm_description/meshes/inspire_hand/left_little_2.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; visual mesh filename=package://rm_description/meshes/inspire_hand/left_little_2.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
- link left_middle_1: geometry collision mesh filename=package://rm_description/meshes/inspire_hand/left_middle_1.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; visual mesh filename=package://rm_description/meshes/inspire_hand/left_middle_1.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
- link left_middle_2: geometry collision mesh filename=package://rm_description/meshes/inspire_hand/left_middle_2.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; visual mesh filename=package://rm_description/meshes/inspire_hand/left_middle_2.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
- link left_ring_1: geometry collision mesh filename=package://rm_description/meshes/inspire_hand/left_ring_1.STL; visual mesh filename=package://rm_description/meshes/inspire_hand/left_ring_1.STL
- link left_ring_2: geometry collision mesh filename=package://rm_description/meshes/inspire_hand/left_ring_2.STL; visual mesh filename=package://rm_description/meshes/inspire_hand/left_ring_2.STL
- link left_thumb_1: geometry collision mesh filename=package://rm_description/meshes/inspire_hand/left_thumb_1.S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; visual mesh filename=package://rm_description/meshes/inspire_hand/left_thumb_1.S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
- link left_thumb_2: geometry collision mesh filename=package://rm_description/meshes/inspire_hand/left_thumb_2.S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; visual mesh filename=package://rm_description/meshes/inspire_hand/left_thumb_2.S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
- link left_thumb_3: geometry collision mesh filename=package://rm_description/meshes/inspire_hand/left_thumb_3.S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; visual mesh filename=package://rm_description/meshes/inspire_hand/left_thumb_3.S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
- link left_thumb_swing: geometry collision mesh filename=package://rm_description/meshes/inspire_hand/left_thumb_swi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; visual mesh filename=package://rm_description/meshes/inspire_hand/left_thumb_swi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
- link robot_base_link: geometry collision mesh filename=package://rm_description/meshes/rm75_6f/base_link_l.STL; visual mesh filename=package://rm_description/meshes/rm75_6f/base_link_l.STL

File: dependence/smart_pick_and_place_ws/src/rm_description/urdf/left_arm_bullet.urdf (robot description, URDF)
Before this commit: robot rm_65_description, 11 links, 10 joints
Links:
- link Link1: geometry collision mesh filename=package://rm_description/meshes/rm75_6f/link1_l.STL; visual mesh filename=package://rm_description/meshes/rm75_6f/link1_l.STL
- link Link2: geometry collision mesh filename=package://rm_description/meshes/rm75_6f/link2_l.STL; visual mesh filename=package://rm_description/meshes/rm75_6f/link2_l.STL
- link Link3: geometry collision mesh filename=package://rm_description/meshes/rm75_6f/link3_l.STL; visual mesh filename=package://rm_description/meshes/rm75_6f/link3_l.STL
- link Link4: geometry collision mesh filename=package://rm_description/meshes/rm75_6f/link4_l.STL; visual mesh filename=package://rm_description/meshes/rm75_6f/link4_l.STL
- link Link5: geometry collision mesh filename=package://rm_description/meshes/rm75_6f/link5_l.STL; visual mesh filename=package://rm_description/meshes/rm75_6f/link5_l.STL
- link Link6: geometry collision mesh filename=package://rm_description/meshes/rm75_6f/link6_l.STL; visual mesh filename=package://rm_description/meshes/rm75_6f/link6_l.STL
- link Link7: geometry collision mesh filename=package://rm_description/meshes/rm75_6f/link7_l.STL; visual mesh filename=package://rm_description/meshes/rm75_6f/link7_l.STL
- link robot_base_link: geometry collision mesh filename=package://rm_description/meshes/rm75_6f/base_link_l.STL; visual mesh filename=package://rm_description/meshes/rm75_6f/base_link_l.STL

File: dependence/smart_pick_and_place_ws/src/rm_description/urdf/right_arm.urdf (robot description, URDF)
Before this commit: robot rm_65_right_description, 22 links, 21 joints
Links:
- link R_Link1: geometry collision mesh filename=package://rm_description/meshes/rm75_6f/link1_l.STL; visual mesh filename=package://rm_description/meshes/rm75_6f/link1_l.STL
- link R_Link2: geometry collision mesh filename=package://rm_description/meshes/rm75_6f/link2_l.STL; visual mesh filename=package://rm_description/meshes/rm75_6f/link2_l.STL
- link R_Link3: geometry collision mesh filename=package://rm_description/meshes/rm75_6f/link3_l.STL; visual mesh filename=package://rm_description/meshes/rm75_6f/link3_l.STL
- link R_Link4: geometry collision mesh filename=package://rm_description/meshes/rm75_6f/link4_l.STL; visual mesh filename=package://rm_description/meshes/rm75_6f/link4_l.STL
- link R_Link5: geometry collision mesh filename=package://rm_description/meshes/rm75_6f/link5_l.STL; visual mesh filename=package://rm_description/meshes/rm75_6f/link5_l.STL
- link R_Link6: geometry collision mesh filename=package://rm_description/meshes/rm75_6f/link6_l.STL; visual mesh filename=package://rm_description/meshes/rm75_6f/link6_l.STL
- link R_Link7: geometry collision mesh filename=package://rm_description/meshes/rm75_6f/link7_l.STL; visual mesh filename=package://rm_description/meshes/rm75_6f/link7_l.STL
- link R_gripper_base: geometry collision mesh filename=package://rm_description/meshes/robotiq_85/robotiq_85_base_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; visual mesh filename=package://rm_description/meshes/robotiq_85/robotiq_85_base_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
- link R_left_inner_finger: geometry collision mesh filename=package://rm_description/meshes/robotiq_85/inner_finger_coa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; visual mesh filename=package://rm_description/meshes/robotiq_85/inner_finger_fin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
- link R_left_inner_knuckle: geometry collision mesh filename=package://rm_description/meshes/robotiq_85/inner_knuckle_co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; visual mesh filename=package://rm_description/meshes/robotiq_85/inner_knuckle_fi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
- link R_left_outer_finger: geometry collision mesh filename=package://rm_description/meshes/robotiq_85/outer_finger_coa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; visual mesh filename=package://rm_description/meshes/robotiq_85/outer_finger_fin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
- link R_left_outer_knuckle: geometry collision mesh filename=package://rm_description/meshes/robotiq_85/outer_knuckle_co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; visual mesh filename=package://rm_description/meshes/robotiq_85/outer_knuckle_fi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
- link R_right_inner_finger: geometry collision mesh filename=package://rm_description/meshes/robotiq_85/inner_finger_coa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; visual mesh filename=package://rm_description/meshes/robotiq_85/inner_finger_fin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
- link R_right_inner_knuckle: geometry collision mesh filename=package://rm_description/meshes/robotiq_85/inner_knuckle_co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; visual mesh filename=package://rm_description/meshes/robotiq_85/inner_knuckle_fi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
- link R_right_outer_finger: geometry collision mesh filename=package://rm_description/meshes/robotiq_85/outer_finger_coa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; visual mesh filename=package://rm_description/meshes/robotiq_85/outer_finger_fin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
- link R_right_outer_knuckle: geometry collision mesh filename=package://rm_description/meshes/robotiq_85/outer_knuckle_co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; visual mesh filename=package://rm_description/meshes/robotiq_85/outer_knuckle_fi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
- link R_robot_base_link: geometry collision mesh filename=package://rm_description/meshes/rm75_6f/base_link_l.STL; visual mesh filename=package://rm_description/meshes/rm75_6f/base_link_l.STL

Commit message: feat: 夹爪上机测试通过，现在可冒烟执行抓取动作

File: dependence/smart_pick_and_place_ws/src/rm_description/urdf/dual_arm.urdf (robot description, URDF)
Before this commit: robot dual_arm, 53 links, 52 joints
Joints:
- joint R_gripper_endeffector_joint: origin xyz=0 0 0.15 rpy=0 0 0 -> xyz=0 0 0.162 rpy=0 0 -1.5708

File: dependence/smart_pick_and_place_ws/src/rm_description/urdf/right_arm.urdf (robot description, URDF)
Before this commit: robot rm_65_right_description, 22 links, 21 joints
Joints:
- joint R_gripper_endeffector_joint: origin xyz=0 0 0.15 rpy=0 0 0 -> xyz=0 0 0.162 rpy=0 0 -1.5708
