Commit message: refactor: 将左臂灵巧手更换为夹爪并进行对应适配，目前左臂抓取仍存在部分偏移待修正

File: dependence/smart_pick_and_place_ws/src/rm_description/urdf/dual_arm.urdf (robot description, URDF)
Before this commit: robot dual_arm, 53 links, 52 joints
Links:
- removed link L_hand_base_link
- removed link L_hand_endeffector
- removed link left_index_1
- removed link left_index_2
- removed link left_little_1
- removed link left_little_2
- removed link left_middle_1
- removed link left_middle_2
- removed link left_ring_1
- removed link left_ring_2
- removed link left_thumb_1
- removed link left_thumb_2
- removed link left_thumb_3
- removed link left_thumb_swing
- added link L_gripper_base, mass 0.30915; collision mesh filename=package://rm_description/meshes/robotiq_85/robotiq_85_base_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; visual mesh filename=package://rm_description/meshes/robotiq_85/robotiq_85_base_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
- added link L_gripper_endeffector, mass 0.0
- added link L_left_inner_finger, mass 0.00724255346165745; collision mesh filename=package://rm_description/meshes/robotiq_85/inner_finger_coa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; visual mesh filename=package://rm_description/meshes/robotiq_85/inner_finger_fin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
- added link L_left_inner_knuckle, mass 0.0110930853895903; collision mesh filename=package://rm_description/meshes/robotiq_85/inner_knuckle_co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; visual mesh filename=package://rm_description/meshes/robotiq_85/inner_knuckle_fi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
- added link L_left_outer_finger, mass 0.0273093985570947; collision mesh filename=package://rm_description/meshes/robotiq_85/outer_finger_coa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; visual mesh filename=package://rm_description/meshes/robotiq_85/outer_finger_fin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
- added link L_left_outer_knuckle, mass 0.00684838849434396; collision mesh filename=package://rm_description/meshes/robotiq_85/outer_knuckle_co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; visual mesh filename=package://rm_description/meshes/robotiq_85/outer_knuckle_fi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
- added link L_right_inner_finger, mass 0.00724255346165744; collision mesh filename=package://rm_description/meshes/robotiq_85/inner_finger_coa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; visual mesh filename=package://rm_description/meshes/robotiq_85/inner_finger_fin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
- added link L_right_inner_knuckle, mass 0.0110930853895903; collision mesh filename=package://rm_description/meshes/robotiq_85/inner_knuckle_co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; visual mesh filename=package://rm_description/meshes/robotiq_85/inner_knuckle_fi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
- added link L_right_outer_finger, mass 0.0273093985570947; collision mesh filename=package://rm_description/meshes/robotiq_85/outer_finger_coa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; visual mesh filename=package://rm_description/meshes/robotiq_85/outer_finger_fin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
- added link L_right_outer_knuckle, mass 0.00684838849401352; collision mesh filename=package://rm_description/meshes/robotiq_85/outer_knuckle_co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; visual mesh filename=package://rm_description/meshes/robotiq_85/outer_knuckle_fi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
Joints:
- removed joint L_hand_joint_endeffector
- removed joint arm_to_hand_virtual
- removed joint left_index_1_joint
- removed joint left_index_2_joint
- removed joint left_little_1_joint
- removed joint left_little_2_joint
- removed joint left_middle_1_joint
- removed joint left_middle_2_joint
- removed joint left_ring_1_joint
- removed joint left_ring_2_joint
- removed joint left_thumb_1_joint
- removed joint left_thumb_2_joint
- removed joint left_thumb_3_joint
- removed joint left_thumb_swing_joint
- added joint L_arm_to_gripper: type fixed, parent Link7, child L_gripper_base, origin xyz=0 0 0.01 rpy=0 0 1.5708, axis 0 0 0
- added joint L_finger_joint: type revolute, parent L_gripper_base, child L_left_outer_knuckle, origin xyz=0.0306011444260539 0 0.0627920162695395 rpy=0 0 0, axis 0 -1 0, limit lower=0 upper=0.725 effort=1000 velocity=2.0
- added joint L_gripper_endeffector_joint: type fixed, parent L_gripper_base, child L_gripper_endeffector, origin xyz=0 0 0.162 rpy=0 0 -1.5708, axis 0 0 0
- added joint L_left_inner_finger_joint: type revolute, parent L_left_inner_knuckle, child L_left_inner_finger, origin xyz=0.034585310861294 0 0.0454970193817975 rpy=0 0 0, axis 0 -1 0, limit lower=0 upper=0.8757 effort=1000 velocity=2.0, mimic joint=L_finger_joint multiplier=-1 offset=0
- added joint L_left_inner_knuckle_joint: type revolute, parent L_gripper_base, child L_left_inner_knuckle, origin xyz=0.0127000000001501 0 0.0693074999999639 rpy=0 0 0, axis 0 -1 0, limit lower=0 upper=0.8757 effort=1000 velocity=2.0, mimic joint=L_finger_joint multiplier=1 offset=0
- added joint L_left_outer_finger_joint: type fixed, parent L_left_outer_knuckle, child L_left_outer_finger, origin xyz=0.0316910442266543 0 -0.00193396375724605 rpy=0 0 0, axis 0 -1 0
- added joint L_right_inner_finger_joint: type revolute, parent L_right_inner_knuckle, child L_right_inner_finger, origin xyz=0.0341060475457406 0 0.0458573878541688 rpy=0 0 0, axis 0 1 0, limit lower=0 upper=0.8757 effort=1000 velocity=2.0, mimic joint=L_finger_joint multiplier=1 offset=0
- added joint L_right_inner_knuckle_joint: type revolute, parent L_gripper_base, child L_right_inner_knuckle, origin xyz=-0.0126999999998499 0 0.0693075000000361 rpy=0 0 3.14159265358979, axis 0 1 0, limit lower=0 upper=0.8757 effort=1000 velocity=2.0, mimic joint=L_finger_joint multiplier=-1 offset=0
- added joint L_right_outer_finger_joint: type fixed, parent L_right_outer_knuckle, child L_right_outer_finger, origin xyz=0.0317095909367246 0 -0.0016013564954687 rpy=0 0 0, axis 0 1 0
- added joint L_right_outer_knuckle_joint: type revolute, parent L_gripper_base, child L_right_outer_knuckle, origin xyz=-0.0306011444258893 0 0.0627920162695395 rpy=0 0 3.14159265358979, axis 0 1 0, limit lower=0 upper=0.8757 effort=1000 velocity=2.0, mimic joint=L_finger_joint multiplier=-1 offset=0

File: dependence/smart_pick_and_place_ws/src/rm_description/urdf/left_arm.urdf (robot description, URDF)
Before this commit: robot rm_65_description, 25 links, 24 joints
Links:
- removed link L_hand_base_link
- removed link L_hand_endeffector
- removed link left_index_1
- removed link left_index_2
- removed link left_little_1
- removed link left_little_2
- removed link left_middle_1
- removed link left_middle_2
- removed link left_ring_1
- removed link left_ring_2
- removed link left_thumb_1
- removed link left_thumb_2
- removed link left_thumb_3
- removed link left_thumb_swing
- added link L_gripper_base, mass 0.30915; collision mesh filename=package://rm_description/meshes/robotiq_85/robotiq_85_base_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; visual mesh filename=package://rm_description/meshes/robotiq_85/robotiq_85_base_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
- added link L_gripper_endeffector, mass 0.0
- added link L_left_inner_finger, mass 0.00724255346165745; collision mesh filename=package://rm_description/meshes/robotiq_85/inner_finger_coa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; visual mesh filename=package://rm_description/meshes/robotiq_85/inner_finger_fin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
- added link L_left_inner_knuckle, mass 0.0110930853895903; collision mesh filename=package://rm_description/meshes/robotiq_85/inner_knuckle_co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; visual mesh filename=package://rm_description/meshes/robotiq_85/inner_knuckle_fi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
- added link L_left_outer_finger, mass 0.0273093985570947; collision mesh filename=package://rm_description/meshes/robotiq_85/outer_finger_coa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; visual mesh filename=package://rm_description/meshes/robotiq_85/outer_finger_fin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
- added link L_left_outer_knuckle, mass 0.00684838849434396; collision mesh filename=package://rm_description/meshes/robotiq_85/outer_knuckle_co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; visual mesh filename=package://rm_description/meshes/robotiq_85/outer_knuckle_fi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
- added link L_right_inner_finger, mass 0.00724255346165744; collision mesh filename=package://rm_description/meshes/robotiq_85/inner_finger_coa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; visual mesh filename=package://rm_description/meshes/robotiq_85/inner_finger_fin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
- added link L_right_inner_knuckle, mass 0.0110930853895903; collision mesh filename=package://rm_description/meshes/robotiq_85/inner_knuckle_co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; visual mesh filename=package://rm_description/meshes/robotiq_85/inner_knuckle_fi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
- added link L_right_outer_finger, mass 0.0273093985570947; collision mesh filename=package://rm_description/meshes/robotiq_85/outer_finger_coa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; visual mesh filename=package://rm_description/meshes/robotiq_85/outer_finger_fin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
- added link L_right_outer_knuckle, mass 0.00684838849401352; collision mesh filename=package://rm_description/meshes/robotiq_85/outer_knuckle_co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; visual mesh filename=package://rm_description/meshes/robotiq_85/outer_knuckle_fi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
Joints:
- removed joint L_hand_joint_endeffector
- removed joint arm_to_hand_virtual
- removed joint left_index_1_joint
- removed joint left_index_2_joint
- removed joint left_little_1_joint
- removed joint left_little_2_joint
- removed joint left_middle_1_joint
- removed joint left_middle_2_joint
- removed joint left_ring_1_joint
- removed joint left_ring_2_joint
- removed joint left_thumb_1_joint
- removed joint left_thumb_2_joint
- removed joint left_thumb_3_joint
- removed joint left_thumb_swing_joint
- added joint L_arm_to_gripper: type fixed, parent Link7, child L_gripper_base, origin xyz=0 0 0.01 rpy=0 0 1.5708, axis 0 0 0
- added joint L_finger_joint: type revolute, parent L_gripper_base, child L_left_outer_knuckle, origin xyz=0.0306011444260539 0 0.0627920162695395 rpy=0 0 0, axis 0 -1 0, limit lower=0 upper=0.725 effort=1000 velocity=2.0
- added joint L_gripper_endeffector_joint: type fixed, parent L_gripper_base, child L_gripper_endeffector, origin xyz=0 0 0.162 rpy=0 0 -1.5708, axis 0 0 0
- added joint L_left_inner_finger_joint: type revolute, parent L_left_inner_knuckle, child L_left_inner_finger, origin xyz=0.034585310861294 0 0.0454970193817975 rpy=0 0 0, axis 0 -1 0, limit lower=0 upper=0.8757 effort=1000 velocity=2.0, mimic joint=L_finger_joint multiplier=-1 offset=0
- added joint L_left_inner_knuckle_joint: type revolute, parent L_gripper_base, child L_left_inner_knuckle, origin xyz=0.0127000000001501 0 0.0693074999999639 rpy=0 0 0, axis 0 -1 0, limit lower=0 upper=0.8757 effort=1000 velocity=2.0, mimic joint=L_finger_joint multiplier=1 offset=0
- added joint L_left_outer_finger_joint: type fixed, parent L_left_outer_knuckle, child L_left_outer_finger, origin xyz=0.0316910442266543 0 -0.00193396375724605 rpy=0 0 0, axis 0 -1 0
- added joint L_right_inner_finger_joint: type revolute, parent L_right_inner_knuckle, child L_right_inner_finger, origin xyz=0.0341060475457406 0 0.0458573878541688 rpy=0 0 0, axis 0 1 0, limit lower=0 upper=0.8757 effort=1000 velocity=2.0, mimic joint=L_finger_joint multiplier=1 offset=0
- added joint L_right_inner_knuckle_joint: type revolute, parent L_gripper_base, child L_right_inner_knuckle, origin xyz=-0.0126999999998499 0 0.0693075000000361 rpy=0 0 3.14159265358979, axis 0 1 0, limit lower=0 upper=0.8757 effort=1000 velocity=2.0, mimic joint=L_finger_joint multiplier=-1 offset=0
- added joint L_right_outer_finger_joint: type fixed, parent L_right_outer_knuckle, child L_right_outer_finger, origin xyz=0.0317095909367246 0 -0.0016013564954687 rpy=0 0 0, axis 0 1 0
- added joint L_right_outer_knuckle_joint: type revolute, parent L_gripper_base, child L_right_outer_knuckle, origin xyz=-0.0306011444258893 0 0.0627920162695395 rpy=0 0 3.14159265358979, axis 0 1 0, limit lower=0 upper=0.8757 effort=1000 velocity=2.0, mimic joint=L_finger_joint multiplier=-1 offset=0

File: dependence/smart_pick_and_place_ws/src/rm_description/urdf/left_arm_bullet.urdf (robot description, URDF)
Before this commit: robot rm_65_description, 11 links, 10 joints
Links:
- added link L_gripper_base, mass 0.30915; collision mesh filename=package://rm_description/meshes/robotiq_85/robotiq_85_base_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; visual mesh filename=package://rm_description/meshes/robotiq_85/robotiq_85_base_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
- added link L_gripper_endeffector, mass 0.0
- added link L_left_inner_finger, mass 0.00724255346165745; collision mesh filename=package://rm_description/meshes/robotiq_85/inner_finger_coa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; visual mesh filename=package://rm_description/meshes/robotiq_85/inner_finger_fin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
- added link L_left_inner_knuckle, mass 0.0110930853895903; collision mesh filename=package://rm_description/meshes/robotiq_85/inner_knuckle_co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; visual mesh filename=package://rm_description/meshes/robotiq_85/inner_knuckle_fi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
- added link L_left_outer_finger, mass 0.0273093985570947; collision mesh filename=package://rm_description/meshes/robotiq_85/outer_finger_coa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; visual mesh filename=package://rm_description/meshes/robotiq_85/outer_finger_fin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
- added link L_left_outer_knuckle, mass 0.00684838849434396; collision mesh filename=package://rm_description/meshes/robotiq_85/outer_knuckle_co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; visual mesh filename=package://rm_description/meshes/robotiq_85/outer_knuckle_fi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
- added link L_right_inner_finger, mass 0.00724255346165744; collision mesh filename=package://rm_description/meshes/robotiq_85/inner_finger_coa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; visual mesh filename=package://rm_description/meshes/robotiq_85/inner_finger_fin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
- added link L_right_inner_knuckle, mass 0.0110930853895903; collision mesh filename=package://rm_description/meshes/robotiq_85/inner_knuckle_co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; visual mesh filename=package://rm_description/meshes/robotiq_85/inner_knuckle_fi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
- added link L_right_outer_finger, mass 0.0273093985570947; collision mesh filename=package://rm_description/meshes/robotiq_85/outer_finger_coa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; visual mesh filename=package://rm_description/meshes/robotiq_85/outer_finger_fin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
- added link L_right_outer_knuckle, mass 0.00684838849401352; collision mesh filename=package://rm_description/meshes/robotiq_85/outer_knuckle_co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; visual mesh filename=package://rm_description/meshes/robotiq_85/outer_knuckle_fi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
Joints:
- added joint L_arm_to_gripper: type fixed, parent Link7, child L_gripper_base, origin xyz=0 0 0.01 rpy=0 0 1.5708, axis 0 0 0
- added joint L_finger_joint: type revolute, parent L_gripper_base, child L_left_outer_knuckle, origin xyz=0.0306011444260539 0 0.0627920162695395 rpy=0 0 0, axis 0 -1 0, limit lower=0 upper=0.725 effort=1000 velocity=2.0
- added joint L_gripper_endeffector_joint: type fixed, parent L_gripper_base, child L_gripper_endeffector, origin xyz=0 0 0.162 rpy=0 0 -1.5708, axis 0 0 0
- added joint L_left_inner_finger_joint: type revolute, parent L_left_inner_knuckle, child L_left_inner_finger, origin xyz=0.034585310861294 0 0.0454970193817975 rpy=0 0 0, axis 0 -1 0, limit lower=0 upper=0.8757 effort=1000 velocity=2.0, mimic joint=L_finger_joint multiplier=-1 offset=0
- added joint L_left_inner_knuckle_joint: type revolute, parent L_gripper_base, child L_left_inner_knuckle, origin xyz=0.0127000000001501 0 0.0693074999999639 rpy=0 0 0, axis 0 -1 0, limit lower=0 upper=0.8757 effort=1000 velocity=2.0, mimic joint=L_finger_joint multiplier=1 offset=0
- added joint L_left_outer_finger_joint: type fixed, parent L_left_outer_knuckle, child L_left_outer_finger, origin xyz=0.0316910442266543 0 -0.00193396375724605 rpy=0 0 0, axis 0 -1 0
- added joint L_right_inner_finger_joint: type revolute, parent L_right_inner_knuckle, child L_right_inner_finger, origin xyz=0.0341060475457406 0 0.0458573878541688 rpy=0 0 0, axis 0 1 0, limit lower=0 upper=0.8757 effort=1000 velocity=2.0, mimic joint=L_finger_joint multiplier=1 offset=0
- added joint L_right_inner_knuckle_joint: type revolute, parent L_gripper_base, child L_right_inner_knuckle, origin xyz=-0.0126999999998499 0 0.0693075000000361 rpy=0 0 3.14159265358979, axis 0 1 0, limit lower=0 upper=0.8757 effort=1000 velocity=2.0, mimic joint=L_finger_joint multiplier=-1 offset=0
- added joint L_right_outer_finger_joint: type fixed, parent L_right_outer_knuckle, child L_right_outer_finger, origin xyz=0.0317095909367246 0 -0.0016013564954687 rpy=0 0 0, axis 0 1 0
- added joint L_right_outer_knuckle_joint: type revolute, parent L_gripper_base, child L_right_outer_knuckle, origin xyz=-0.0306011444258893 0 0.0627920162695395 rpy=0 0 3.14159265358979, axis 0 1 0, limit lower=0 upper=0.8757 effort=1000 velocity=2.0, mimic joint=L_finger_joint multiplier=-1 offset=0

Commit message: refactor: 劳朱ddl冲刺base版本

File: dependence/smart_pick_and_place_ws/src/rm_description/urdf/dual_arm.urdf (robot description, URDF)
Before this commit: robot dual_arm, 49 links, 48 joints
Links:
- removed link R_cam_link_grasp
Joints:
- removed joint R_cam_link_grasp_joint
- joint base_to_R_base: origin xyz=0.99 -0.72 0 rpy=0 0 1.5708 -> xyz=0.35 -0.71 0 rpy=0 0 1.5708

File: dependence/smart_pick_and_place_ws/src/rm_description/urdf/right_arm.urdf (robot description, URDF)
Before this commit: robot rm_65_right_description, 22 links, 21 joints
Links:
- removed link R_cam_link_grasp
Joints:
- removed joint R_cam_link_grasp_joint
